File: KiCad/IBM_5324_Keyboard.kicad_pcb (KiCad board)
At the start: 2 copper layers, 423 x 116 mm, 85 parts, among them SW1 CMD, SW10 ERASE, SW11 | 1, SW12 # 3, SW13 % 5, SW14 & 7, SW15 * +, SW16 ( 9, SW17 _ -, SW18 RH <-, SW19 / -, SW2 ~ `, SW20 NP 8, SW21 HOLD, SW22 FIELD ADV, SW23 W, SW24 R, SW25 Y, SW26 I, SW27 P, SW28 | \, SW29 NP 7, SW3 @ 2, SW30 NP 9, SW31 INQ, SW32 SHIFT LOCK, SW33 Q, SW34 E, SW35 T, SW36 O, SW37 ! ¢, SW38 ENTER, SW39 NP 4, SW4 $ 4, SW40 FIELD-, SW41 U, SW42 ERROR RESET, SW43 LH SHIFT, SW44 A, SW45 D, SW46 G, SW47 J, SW48 L, SW49 " ', SW5 ^ 6, SW50 } {, SW51 NP 5, SW52 NP 6, SW53 TEST, SW54 SCROLL DOWN, SW55 S, SW56 F, SW57 H, SW58 SCROLL UP, SW59 K, SW6 * 8, SW60 : ;, SW61 NEWLINE, SW62 NP 1, SW63 NP 3, SW64 ->, SW65 > <, SW66 C, SW67 B, SW68 M, SW69 . ., SW7 ) 0, SW70 RH SHIFT, SW71 NP 2, SW72 FIELD+, SW73 N, SW74 LH <-, SW75 ALT, SW76 Z, SW77 X, SW78 V, SW79 SPACE, SW8 + =, SW80 , ,, SW81 ? /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

Commit message: Update IBM_5324_Keyboard.kicad_pcb
Connections:
- SW58 pad 2: Row_6 -> Row_7
- SW64 pad 2: Row_6 -> Row_7
- SW65 pad 2: Row_6 -> Row_7
- SW66 pad 2: Row_6 -> Row_7
- SW67 pad 2: Row_6 -> Row_7
- SW68 pad 2: Row_6 -> Row_7
- SW69 pad 2: Row_6 -> Row_7
- SW70 pad 2: Row_6 -> Row_7
- SW71 pad 2: Row_6 -> Row_7
- SW72 pad 2: Row_6 -> Row_7
- SW73 pad 2: Row_6 -> Row_7
- SW74 pad 2: Row_6 -> Row_8
- SW75 pad 2: Row_6 -> Row_8
- SW76 pad 2: Row_6 -> Row_8
- SW77 pad 2: Row_6 -> Row_8
- SW78 pad 2: Row_6 -> Row_8
- SW79 pad 2: Row_6 -> Row_8
- SW80 pad 2: Row_6 -> Row_8
- SW81 pad 2: Row_6 -> Row_8
- SW82 pad 2: Row_6 -> Row_8
- SW83 pad 2: Row_6 -> Row_8
- SW84 pad 2: Row_6 -> Row_8
Changed lines of the file:
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@@
 	(net 16 "Row_5")
 	(net 17 "Row_6")
+	(net 18 "Row_7")
+	(net 19 "Row_8")
 	(footprint "PCM_Switch_Keyboard_Cherry_MX:SW_Cherry_MX_PCB"
 		(layer "F.Cu")
@@
 			(layers "*.Cu" "*.Mask")
 			(remove_unused_layers no)
-			(net 17 "Row_6")
+			(net 18 "Row_7")
 			(pinfunction "2")
 			(pintype "passive")
@@
 			(layers "*.Cu" "*.Mask")
 			(remove_unused_layers no)
-			(net 17 "Row_6")
+			(net 18 "Row_7")
 			(pinfunction "2")
 			(pintype "passive")
@@
 			(layers "*.Cu" "*.Mask")
 			(remove_unused_layers no)
-			(net 17 "Row_6")
+			(net 19 "Row_8")
 			(pinfunction "2")
 			(pintype "passive")
@@
 			(layers "*.Cu" "*.Mask")
 			(remove_unused_layers no)
-			(net 17 "Row_6")
+			(net 19 "Row_8")
 			(pinfunction "2")
 			(pintype "passive")
@@
 			(layers "*.Cu" "*.Mask")
 			(remove_unused_layers no)
-			(net 17 "Row_6")
+			(net 18 "Row_7")
 			(pinfunction "2")
 			(pintype "passive")
@@
 			(layers "*.Cu" "*.Mask")
 			(remove_unused_layers no)
-			(net 17 "Row_6")
+			(net 19 "Row_8")
 			(pinfunction "2")
 			(pintype "passive")
@@
 			(layers "*.Cu" "*.Mask")
 			(remove_unused_layers no)
-			(net 17 "Row_6")
+			(net 19 "Row_8")
 			(pinfunction "2")
 			(pintype "passive")
@@
 			(layers "*.Cu" "*.Mask")
 			(remove_unused_layers no)
-			(net 17 "Row_6")
+			(net 19 "Row_8")
 			(pinfunction "2")
 			(pintype "passive")
@@
 			(layers "*.Cu" "*.Mask")
 			(remove_unused_layers no)
-			(net 17 "Row_6")
+			(net 18 "Row_7")
 			(pinfunction "2")
 			(pintype "passive")
@@
 			(layers "*.Cu" "*.Mask")
 			(remove_unused_layers no)
-			(net 17 "Row_6")
+			(net 18 "Row_7")
 			(pinfunction "2")
 			(pintype "passive")
@@
 			(layers "*.Cu" "*.Mask")
 			(remove_unused_layers no)
-			(net 17 "Row_6")
+			(net 19 "Row_8")
 			(pinfunction "2")
 			(pintype "passive")
@@
 			(layers "*.Cu" "*.Mask")
 			(remove_unused_layers no)
-			(net 17 "Row_6")
+			(net 18 "Row_7")
 			(pinfunction "2")
 			(pintype "passive")
@@
 			(layers "*.Cu" "*.Mask")
 			(remove_unused_layers no)
-			(net 17 "Row_6")
+			(net 19 "Row_8")
 			(pinfunction "2")
 			(pintype "passive")
@@
 			(layers "*.Cu" "*.Mask")
 			(remove_unused_layers no)
-			(net 17 "Row_6")
+			(net 18 "Row_7")
 			(pinfunction "2")
 			(pintype "passive")
@@
 			(layers "*.Cu" "*.Mask")
 			(remove_unused_layers no)
-			(net 17 "Row_6")
+			(net 18 "Row_7")
 			(pinfunction "2")
 			(pintype "passive")
@@
 			(layers "*.Cu" "*.Mask")
 			(remove_unused_layers no)
-			(net 17 "Row_6")
+			(net 19 "Row_8")
 			(pinfunction "2")
 			(pintype "passive")
@@
 			(layers "*.Cu" "*.Mask")
 			(remove_unused_layers no)
-			(net 17 "Row_6")
+			(net 18 "Row_7")
 			(pinfunction "2")
 			(pintype "passive")
@@
 			(layers "*.Cu" "*.Mask")
 			(remove_unused_layers no)
-			(net 17 "Row_6")
+			(net 19 "Row_8")
 			(pinfunction "2")
 			(pintype "passive")
@@
 			(layers "*.Cu" "*.Mask")
 			(remove_unused_layers no)
-			(net 17 "Row_6")
+			(net 18 "Row_7")
 			(pinfunction "2")
 			(pintype "passive")
@@
 			(layers "*.Cu" "*.Mask")
 			(remove_unused_layers no)
-			(net 17 "Row_6")
+			(net 19 "Row_8")
 			(pinfunction "2")
 			(pintype "passive")
@@
 			(layers "*.Cu" "*.Mask")
 			(remove_unused_layers no)
-			(net 17 "Row_6")
+			(net 19 "Row_8")
 			(pinfunction "2")
 			(pintype "passive")
@@
 			(layers "*.Cu" "*.Mask")
 			(remove_unused_layers no)
-			(net 17 "Row_6")
+			(net 18 "Row_7")
 			(pinfunction "2")
 			(pintype "passive")
@@
 		(layer "Edge.Cuts")
 	)
+	(gr_text "WORK IN PROGRESS"
+		(at 260.84515 181.2924 0)
+		(layer "F.SilkS")
+		(effects
+			(font
+				(size 5 5)
+				(thickness 0.3)
+				(bold yes)
+			)
+			(justify left bottom)
+		)
+	)
 	(gr_text "IBM 5324 Datamaster Keyboard\nBrett Hallen, Nov 2025"

Commit message: Progressing design
Parts:
- added J1: To 5324, Clueless_Engineer:L77SDB25SA4CH4F, F.Cu at (442.9, 167.5)
- added J2: Conn_02x14_Row_Letter_First, Connector_PinHeader_2.54mm:PinHeader_2x14_P2.54mm_Vertical, F.Cu at (442.9, 175.3)
Routing:
- net Col_B: track 0.00 -> 163.7 mm
- net Col_C: track 0.00 -> 145.5 mm
- net Col_D: track 0.00 -> 144.2 mm
- net Col_E: track 0.00 -> 144.2 mm
- net Col_G: track 0.00 -> 143.2 mm
- net Col_H: track 0.00 -> 143.2 mm
- net Col_J: track 0.00 -> 141.4 mm
- net Col_A: track 0.00 -> 133.4 mm
- net Col_K: track 0.00 -> 122.2 mm
- net Row_4: track 433.3 -> 333.1 mm
- net Col_F: track 0.00 -> 94.1 mm
- net +12V: track 0.00 -> 30.1 mm
- net PROGRAM RESET: track 0.00 -> 18.9 mm
- net DELAY STROBE: track 0.00 -> 16.5 mm
- net SCAN CODE BIT 0: track 0.00 -> 14.2 mm
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Other:
- board size 423 x 116 mm -> 419.1 x 128.3 mm
- board text added: "IBM System/23 Datamaster Model 5324 Keyboard Brett Hallen, Nov 2025"
- board text removed: "IBM 5324 Datamaster Keyboard Brett Hallen, Nov 2025"

Commit message: Key switch routing completed
Parts:
- added H1: MountingHole, MountingHole:MountingHole_3.2mm_M3, F.Cu at (68.2, 159.6)
- added H2: MountingHole, MountingHole:MountingHole_3.2mm_M3, F.Cu at (68.2, 285.6)
- added H3: MountingHole, MountingHole:MountingHole_3.2mm_M3, F.Cu at (209.2, 159.6)
- added H4: MountingHole, MountingHole:MountingHole_3.2mm_M3, F.Cu at (209.2, 285.6)
- added H5: MountingHole, MountingHole:MountingHole_3.2mm_M3, F.Cu at (350.2, 159.6)
- added H6: MountingHole, MountingHole:MountingHole_3.2mm_M3, F.Cu at (350.2, 285.6)
- added H7: MountingHole, MountingHole:MountingHole_3.2mm_M3, F.Cu at (491.2, 159.6)
- added H8: MountingHole, MountingHole:MountingHole_3.2mm_M3, F.Cu at (491.2, 285.6)
- J2: value Conn_02x14_Row_Letter_First -> To DB25; footprint Connector_PinHeader_2.54mm:PinHeader_2x14_P2.54mm_Vertical -> Connector_PinHeader_2.54mm:PinHeader_2x08_P2.54mm_Vertical
- moved J2 0.69 mm to (443.2, 175.9)
Routing:
- net Row_7: track 0.00 -> 419.4 mm
- net Row_8: track 0.00 -> 404.0 mm
- net Row_5: track 0.00 -> 400.3 mm
- net Row_6: track 0.00 -> 393.9 mm
- net Col_I: track 0.00 -> 139.2 mm
- net Row_4: track 333.1 -> 433.3 mm
- net +12V: track 30.1 -> 37.0 mm
- net DELAY STROBE: track 16.5 -> 12.8 mm
- net SCAN CODE BIT 0: track 14.2 -> 17.5 mm
- net SCAN CODE BIT 4: track 11.1 -> 14.1 mm
- net SCAN CODE BIT 3: track 9.33 -> 12.4 mm
- net DATA STROBE: track 5.24 -> 8.09 mm
- net SCAN CODE BIT 5: track 7.25 -> 10.1 mm
- net SCAN CODE BIT 2: track 12.2 -> 15.0 mm
- net Row_3: track 369.0 -> 366.5 mm, vias 1 -> 0
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- added copper zone on B.Cu, net GND
- added copper zone on F.Cu, net GND
Other:
- board size 419.1 x 128.3 mm -> 431 x 134 mm
- board text added: "A1"
- board text added: "A2"
- board text added: "A3"
- board text added: "A4"
- board text added: "A5"
- board text added: "A6"
- board text added: "A7"
- board text added: "A8"
- board text added: "B1"
- board text added: "B3"
- board text added: "B4"
- board text added: "B5"
- board text added: "B6"
- board text added: "B7"
- board text added: "B8"

Commit message: Started work on firmware
Parts:
- added U1: ATmega2560-16A, Package_QFP:TQFP-100_14x14mm_P0.5mm, F.Cu at (391.1, 168.3)

Commit message: Started firmware development
Parts:
- added U2: LM7805_TO220, Package_TO_SOT_THT:TO-220-3_Horizontal_TabDown, F.Cu at (471.1, 175.9)
- U1: value ATmega2560-16A -> Teensy4.1; footprint Package_QFP:TQFP-100_14x14mm_P0.5mm -> Clueless_Engineer:Teensy41
- moved U1 11.4 mm to (380.9, 173.4), turned to 180 degrees
Connections:
- U1 pad 1: unconnected-(U1-PG5-Pad1) -> GND
- U1 pad 10: Net-(U1-VCC-Pad10) -> unconnected-(U1-8_TX2_IN1-Pad10)
- U1 pad 11: Net-(U1-GND-Pad11) -> unconnected-(U1-9_OUT1C-Pad11)
- U1 pad 31: Net-(U1-VCC-Pad10) -> unconnected-(U1-39_MISO1_OUT1A-Pad31)
- U1 pad 32: Net-(U1-GND-Pad11) -> unconnected-(U1-40_A16-Pad32)
- U1 pad 34: unconnected-(U1-XTAL1-Pad34) -> GND
- U1 pad 48: unconnected-(U1-PD5-Pad48) -> +5V
- U1 pad 52: unconnected-(U1-PG1-Pad52) -> GND
- U1 pad 58: unconnected-(U1-PC5-Pad58) -> GND
- U1 pad 59: unconnected-(U1-PC6-Pad59) -> GND
- U1 pad 61: Net-(U1-VCC-Pad10) -> unconnected-(U1-LED-Pad61)
- U1 pad 62: Net-(U1-GND-Pad11) -> unconnected-(U1-T--Pad62)
- U1 pad 64: unconnected-(U1-PJ1-Pad64) -> GND
Routing:
- net +5V: track 0.00 -> 61.0 mm
- net +12V: track 37.0 -> 62.0 mm
