File: KiCad/IBM_5324_Keyboard.kicad_pcb (KiCad board)
At the start: 2 copper layers, 431 x 134 mm, 99 parts, among them J1 To 5324, J2 To DB25, SW1 CMD, SW10 ERASE, SW11 | 1, SW12 # 3, SW13 % 5, SW14 & 7, SW15 * +, SW16 ( 9, SW17 _ -, SW18 RH <-, SW19 / -, SW2 ~ `, SW20 NP 8, SW21 HOLD, SW22 FIELD ADV, SW23 W, SW24 R, SW25 Y, SW26 I, SW27 P, SW28 | \, SW29 NP 7, SW3 @ 2, SW30 NP 9, SW31 INQ, SW32 SHIFT LOCK, SW33 Q, SW34 E, SW35 T, SW36 O, SW37 ! ¢, SW38 ENTER, SW39 NP 4, SW4 $ 4, SW40 FIELD-, SW41 U, SW42 ERROR RESET, SW43 LH SHIFT, SW44 A, SW45 D, SW46 G, SW47 J, SW48 L, SW49 " ', SW5 ^ 6, SW50 } {, SW51 NP 5, SW52 NP 6, SW53 TEST, SW54 SCROLL DOWN, SW55 S, SW56 F, SW57 H, SW58 SCROLL UP, SW59 K, SW6 * 8, SW60 : ;, SW61 NEWLINE, SW62 NP 1, SW63 NP 3, SW64 ->, SW65 > <, SW66 C, SW67 B, SW68 M, SW69 . ., SW7 ) 0, SW70 RH SHIFT, SW71 NP 2, SW72 FIELD+, SW73 N, SW74 LH <-, SW75 ALT, SW76 Z, SW77 X, SW78 V, SW79 SPACE, SW8 + =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

Commit message: Design tweaks
Parts:
- U3: footprint Package_DIP:DIP-18_W7.62mm -> Package_DIP:DIP-20_W7.62mm
- moved C1 20.3 mm to (435.3, 181.0)
- moved U2 2.84 mm to (489.9, 178.4), turned to 180 degrees
- moved H1 1.00 mm to (68.2, 160.6)
- moved H3 1.00 mm to (209.2, 160.6)
- moved H5 1.00 mm to (350.2, 160.6)
- moved H7 1.00 mm to (491.2, 160.6)
- renumbered SW16 to SW15, SW17 to SW16, SW18 to SW17, SW20 to SW18, SW21 to SW20, SW22 to SW21, SW23 to SW22, SW24 to SW23, SW25 to SW24, SW26 to SW25, SW27 to SW26, SW28 to SW27, SW29 to SW28, SW30 to SW29, SW31 to SW30, SW32 to SW31, SW33 to SW32, SW34 to SW33, SW35 to SW34, SW41 to SW35, SW42 to SW41, SW43 to SW42, SW44 to SW43, SW45 to SW44, SW46 to SW45, SW47 to SW46, SW48 to SW47, SW49 to SW48, SW50 to SW49, SW51 to SW50, SW52 to SW51, SW53 to SW52, SW54 to SW53, SW55 to SW54, SW56 to SW55, SW57 to SW56, SW59 to SW57, SW60 to SW58, SW61 to SW59, SW62 to SW60, SW63 to SW61, SW58 to SW62, SW64 to SW63, SW65 to SW64, SW66 to SW65, SW67 to SW66, SW73 to SW67, SW74 to SW73, SW75 to SW74, SW76 to SW75, SW77 to SW76, SW78 to SW77, SW79 to SW78, SW80 to SW79, SW81 to SW80, SW82 to SW81, SW83 to SW82, SW84 to SW83, SW15 to SW9
Connections:
- net DATA STROBE_{BUFF} renamed DATA STROB~{E}
- net SCAN CODE BIT 0_{BUFF} renamed SCAN CODE BIT ~{0}
- net SCAN CODE BIT 1_{BUFF} renamed SCAN CODE BIT ~{1}
- net SCAN CODE BIT 2_{BUFF} renamed SCAN CODE BIT ~{2}
- net SCAN CODE BIT 3_{BUFF} renamed SCAN CODE BIT ~{3}
- net SCAN CODE BIT 4_{BUFF} renamed SCAN CODE BIT ~{4}
- net SCAN CODE BIT 5_{BUFF} renamed SCAN CODE BIT ~{5}
- net SCAN CODE BIT 6_{BUFF} renamed SCAN CODE BIT ~{6}
- U1 pad 47: unconnected-(U1-GND-Pad47) -> GND
- U1 pad 52: GND -> unconnected-(U1-GND-Pad52)
- U1 pad 58: GND -> unconnected-(U1-GND-Pad58)
- U1 pad 59: GND -> unconnected-(U1-GND-Pad59)
- U1 pad 64: GND -> unconnected-(U1-GND-Pad64)
Routing:
- net +5V: track 109.1 -> 134.0 mm
- net SCAN CODE BIT ~{4}: track 41.2 -> 44.6 mm
- net SCAN CODE BIT ~{6}: track 36.6 -> 38.7 mm
- net SCAN CODE BIT ~{3}: track 42.8 -> 44.7 mm
- net SCAN CODE BIT ~{1}: track 44.0 -> 45.8 mm
- net Col_C: track 321.6 -> 319.8 mm
- net DATA STROB~{E}: track 30.8 -> 29.2 mm
- net SCAN CODE BIT ~{0}: track 45.0 -> 46.4 mm
- net SCAN CODE BIT ~{2}: track 43.3 -> 44.6 mm
- net SCAN CODE BIT ~{5}: track 41.2 -> 40.5 mm
- net GND: vias 39 -> 50
Other:
- board size 431 x 134 mm -> 437 x 133 mm

Commit message: Swapped DB25 female to male
Parts:
- added D1: +5V, LED_THT:LED_D5.0mm, F.Cu at (402.3, 160.6)
- added R1: R, Resistor_THT:R_Axial_DIN0207_L6.3mm_D2.5mm_P7.62mm_Horizontal, F.Cu at (416.3, 160.6)
- J1: footprint Clueless_Engineer:L77SDB25SA4CH4F -> Clueless_Engineer:L717SDB25P1ACH3R
- moved J2 32.8 mm to (475.5, 176.9), turned to -90 degrees
- moved J1 32.6 mm to (475.5, 169.6)
- moved C1 19.5 mm to (415.8, 180.7)
Connections:
- U1 pad 12: DELAY STROBE -> PROGRAM RESET
- U1 pad 13: PROGRAM RESET -> DELAY STROBE
Routing:
- net DATA STROB~{E}: track 29.2 -> 61.2 mm
- net +12V: track 38.9 -> 63.6 mm
- net +5V: track 134.0 -> 110.2 mm
- net SCAN CODE BIT ~{6}: track 38.7 -> 55.9 mm
- net PROGRAM RESET: track 103.9 -> 88.7 mm
- net SCAN CODE BIT ~{5}: track 40.5 -> 54.0 mm
- net SCAN CODE BIT ~{4}: track 44.6 -> 52.0 mm
- net SCAN CODE BIT ~{3}: track 44.7 -> 50.1 mm
- net Net-(D1-A): track 0.00 -> 3.81 mm
- net SCAN CODE BIT ~{2}: track 44.6 -> 48.2 mm
- net DELAY STROBE: track 96.5 -> 93.9 mm
- net SCAN CODE BIT ~{0}: track 46.4 -> 45.1 mm
- net SCAN CODE BIT ~{1}: track 45.8 -> 47.0 mm
- net GND: vias 50 -> 23
Other:
- board text added: "(ALL GROUND/RETURN THIS SIDE) A1"
- board text removed: "A1 (ALL GROUND/RETURN THIS SIDE)"
- board text removed: "B10"
- board text removed: "WORK IN PROGRESS"

Commit message: Added external pull-up array on rows
Parts:
- added RN1: 4.7KΩ, Resistor_THT:R_Array_SIP9, F.Cu at (403.8, 184.8)
- D1: value +5V -> +5V Power
Routing:
- net +5V: track 110.2 -> 118.2 mm
- net Row_1: track 390.1 -> 397.7 mm
- net Row_2: track 430.3 -> 431.5 mm
- net GND: vias 23 -> 46

Commit message: Revised schematic & PCB layout
Parts:
- added D2: +12V, LED_THT:LED_D5.0mm, F.Cu at (394.7, 160.6)
- added R2: R, Resistor_THT:R_Axial_DIN0207_L6.3mm_D2.5mm_P7.62mm_Horizontal, F.Cu at (416.3, 160.6)
- D1: value +5V Power -> +5V
- SW70: footprint PCM_Switch_Keyboard_Cherry_MX:SW_Cherry_MX_PCB -> PCM_Switch_Keyboard_Cherry_MX:SW_Cherry_MX_PCB_1.50u
- moved U1 87.9 mm to (293.1, 172.1)
- moved U2 75.1 mm to (415.0, 173.3), turned to 0 degrees
- moved RN1 38.1 mm to (374.3, 160.6), turned to -90 degrees
- moved C1 13.7 mm to (402.3, 178.4), turned to 90 degrees
- moved R1 3.81 mm to (416.3, 164.5)
Connections:
- net +12V renamed /+12V
- net +5V renamed /+5V
- net DATA STROBE renamed /DS
- net DATA STROB~{E} renamed /DATA STROBE
- net DELAY STROBE renamed /DELAY STROBE
- net GND renamed /GND
- net PROGRAM RESET renamed /PROGRAM RESET
- net SCAN CODE BIT 0 renamed /SCB_{0}
- net SCAN CODE BIT 1 renamed /SCB1
- net SCAN CODE BIT 2 renamed /SCB2
- net SCAN CODE BIT 3 renamed /SCB3
- net SCAN CODE BIT 4 renamed /SCB4
- net SCAN CODE BIT 5 renamed /SCB5
- net SCAN CODE BIT 6 renamed /SCB6
- net SCAN CODE BIT ~{0} renamed /SCAN CODE BIT 0
- net SCAN CODE BIT ~{1} renamed /SCAN CODE BIT 1
- net SCAN CODE BIT ~{2} renamed /SCAN CODE BIT 2
- net SCAN CODE BIT ~{3} renamed /SCAN CODE BIT 3
- net SCAN CODE BIT ~{4} renamed /SCAN CODE BIT 4
- net SCAN CODE BIT ~{5} renamed /SCAN CODE BIT 5
- net SCAN CODE BIT ~{6} renamed /SCAN CODE BIT 6
Routing:
- net Col_A: track 418.0 -> 311.6 mm
- net Row_8: track 591.5 -> 694.5 mm
- net Row_7: track 571.7 -> 672.9 mm
- net Row_6: track 553.9 -> 653.4 mm
- net Row_5: track 541.6 -> 639.3 mm
- net Row_4: track 545.1 -> 641.0 mm
- net Row_3: track 481.8 -> 575.9 mm
- net Row_2: track 431.5 -> 523.9 mm
- net Col_K: track 227.0 -> 319.1 mm
- net Col_J: track 210.9 -> 302.5 mm
- net /SCB5: track 35.5 -> 126.7 mm
- net /SCB6: track 38.0 -> 127.8 mm
- net /DELAY STROBE: track 93.9 -> 182.5 mm
- net Col_I: track 175.2 -> 263.6 mm
- net /DS: track 41.6 -> 130.0 mm
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Other:
- board text added: "+12V"
- board text added: "+5V"
- board text added: "1.25u"
- board text added: "1.5u"
- board text added: "1.75u"
- board text added: "2u"
- board text added: "3u"
- board text added: "DB25 Male"
