File: KiCad/IBM_5324_Keyboard.kicad_pcb (KiCad board)
At the start: 2 copper layers, 437 x 133 mm, 107 parts, among them J1 To 5324, J2 To DB25, SW1 CMD, SW10 ERASE, SW11 | 1, SW12 # 3, SW13 % 5, SW14 & 7, SW15 ( 9, SW16 _ -, SW17 RH <-, SW18 NP 8, SW19 / -, SW2 ~ `, SW20 HOLD, SW21 FIELD ADV, SW22 W, SW23 R, SW24 Y, SW25 I, SW26 P, SW27 | \, SW28 NP 7, SW29 NP 9, SW3 @ 2, SW30 INQ, SW31 SHIFT LOCK, SW32 Q, SW33 E, SW34 T, SW35 U, SW36 O, SW37 ! ¢, SW38 ENTER, SW39 NP 4, SW4 $ 4, SW40 FIELD-, SW41 ERROR RESET, SW42 LH SHIFT, SW43 A, SW44 D, SW45 G, SW46 J, SW47 L, SW48 " ', SW49 } {, SW5 ^ 6, SW50 NP 5, SW51 NP 6, SW52 TEST, SW53 SCROLL DOWN, SW54 S, SW55 F, SW56 H, SW57 K, SW58 : ;, SW59 NEWLINE, SW6 * 8, SW60 NP 1, SW61 NP 3, SW62 SCROLL UP, SW63 ->, SW64 > <, SW65 C, SW66 B, SW67 N, SW68 M, SW69 . ., SW7 ) 0, SW70 RH SHIFT, SW71 NP 2, SW72 FIELD+, SW73 LH <-, SW74 ALT, SW75 Z, SW76 X, SW77 V, SW78 SPACE, SW79 , ,, SW8 + =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

Commit message: Further refinements to PCB layout
- missing value text on some parts
- isolated ground on 74LS245
Connections:
- net /DATA STROBE renamed /~{DATA STROBE_{B}}
- net /DELAY STROBE renamed /~{DELAY STROBE}
- net /DELAY STROB~{E} renamed /~{DELAY STROBE_{B}}
- net /DS renamed /~{DATA STROBE}
- net /PROGRAM RESET renamed /~{PROGRAM RESET}
- net /PROGRAM RESE~{T} renamed /~{PROGRAM RESET_{B}}
- net /SCAN CODE BIT 0 renamed /~{SCAN CODE BIT 0_{B}}
- net /SCAN CODE BIT 1 renamed /~{SCAN CODE BIT 1_{B}}
- net /SCAN CODE BIT 2 renamed /~{SCAN CODE BIT 2_{B}}
- net /SCAN CODE BIT 3 renamed /~{SCAN CODE BIT 3_{B}}
- net /SCAN CODE BIT 4 renamed /~{SCAN CODE BIT 4_{B}}
- net /SCAN CODE BIT 5 renamed /~{SCAN CODE BIT 5_{B}}
- net /SCAN CODE BIT 6 renamed /~{SCAN CODE BIT 6_{B}}
- net /SCB1 renamed /~{SCAN CODE BIT 1}
- net /SCB2 renamed /~{SCAN CODE BIT 2}
- net /SCB3 renamed /~{SCAN CODE BIT 3}
- net /SCB4 renamed /~{SCAN CODE BIT 4}
- net /SCB5 renamed /~{SCAN CODE BIT 5}
- net /SCB6 renamed /~{SCAN CODE BIT 6}
- net /SCB_{0} renamed /~{SCAN CODE BIT 0}
Routing:
- net /GND: vias 19 -> 42
- net (no net): vias 0 -> 1
Other:
- board text added: "Designed in Port Macquarie, Australia"
- board text added: "IBM System/23 Datamaster Model 5324 Keyboard (Rev. A) Brett Hallen, Nov 2025"
- board text removed: "IBM System/23 Datamaster Model 5324 Keyboard Brett Hallen, Nov 2025"
